Commit message: 2 jun

File: Basics of pyBullet/Week 1/Subpart 2/robourdfcode.urdf (robot description, URDF)
Before this commit: robot 2_R_robot, 2 links, 1 joints
Links:
- added link link_2; visual cylinder length=1.5 radius=0.03
- added link palm; visual box size=0.3 0.3 0.3
- link fixed_base: geometry visual box size=0 0 0
- link link_1: geometry visual cylinder length=1.5 radius=0.03
Joints:
- added joint Revolute_joint_2: type revolute, parent link_1, child link_2, origin xyz=1.5 0 0 rpy=0 0 0, axis 0 1 0, limit lower=-3.14 upper=3.14 effort=1000.0 velocity=0.5
- added joint palm_joint: type fixed, parent link_2, child palm, origin xyz=1.5 0 0 rpy=0 0 0, axis 0 1 0
- joint Revolute_joint_1: axis 0 0 1 -> 0 1 0
