Commit message: jun 3

File: Basics of pyBullet/Week 1/Subpart 3/sphere.urdf (robot description, URDF)
Before this commit: robot sphere, 1 links, 0 joints
Links:
- link base: geometry collision sphere radius=2; visual sphere radius=2

Commit message: jun 3

File: Basics of pyBullet/Week 1/Subpart 3/sphere.urdf (robot description, URDF)
Before this commit: robot sphere, 1 links, 0 joints
Links:
- link base: geometry collision sphere radius=0.01; visual sphere radius=0.03

Commit message: final submissions for week 1

File: Basics of pyBullet/Week 1/Subpart 3/sphere.urdf (robot description, URDF)
Before this commit: robot sphere, 1 links, 0 joints
Links:
- link base: geometry collision sphere radius=0.05; visual sphere radius=0.05
